File: schematics/venabili.sch (KiCad schematic (older format))
At the start: 96 parts

Commit message: Schematics: Add MCU
Parts:
- added U?: STM32F103C8Tx, Housings_QFP:LQFP-48_7x7mm_Pitch0.5mm, symbol STM32F103C8Tx
Connections:
- net labels added: A1, A10, A11, A12, A2, A3, A4, A5, A6, A7, A8, A9, B5, B6, B7, B8
- wire segments 12 -> 64
Other:
- moved on the sheet: D?, SW?

Commit message: Finish schematics
Parts:
- removed U?: STM32F103C8Tx, Housings_QFP:LQFP-48_7x7mm_Pitch0.5mm, symbol STM32F103C8Tx
- added J1: USB_B_Mini, symbol Connector:USB_B_Mini
- D1, D10, D11, D12, D13, D14, D15, D16, D17, D18, D19, D2, D20, D21, D22, D23, D24, D25, D26, D27, D28, D29, D3, D30, D31, D32, D33, D34, D35, D36, D37, D38, D39, D4, D40, D41, D42, D43, D44, D45, D46, D47, D48, D5, D6, D7, D8, D9: renamed from D?; symbol D -> venabili-rescue:D
- SW1, SW10, SW11, SW12, SW13, SW14, SW15, SW16, SW17, SW18, SW19, SW2, SW20, SW21, SW22, SW23, SW24, SW25, SW26, SW27, SW28, SW29, SW3, SW30, SW31, SW32, SW33, SW34, SW35, SW36, SW37, SW38, SW39, SW4, SW40, SW41, SW42, SW43, SW44, SW45, SW46, SW47, SW48, SW5, SW6, SW7, SW8, SW9: renamed from SW?; symbol SW_Push -> venabili-rescue:SW_Push
Connections:
- net B5 is gone; now on net B6: SW1.2, SW13.2, SW17.2, SW21.2, SW25.2, SW29.2, SW33.2, SW37.2, SW41.2, SW45.2, SW5.2, SW9.2
- net A1: now also D5.1 (K), D6.1 (K), D7.1 (K), D8.1 (K); no longer D4.1 (K)
- net A10: now also D41.1 (K), D42.1 (K), D43.1 (K), D44.1 (K); no longer D40.1 (K)
- net A11: now also D45.1 (K), D46.1 (K), D47.1 (K), D48.1 (K), J1.2 (D-); no longer D44.1 (K)
- net A12: now also J1.3 (D+); no longer D48.1 (K)
- net A2: now also D10.1 (K), D11.1 (K), D12.1 (K), D9.1 (K); no longer D8.1 (K)
- net A3: now also D13.1 (K), D14.1 (K), D15.1 (K), D16.1 (K); no longer D12.1 (K)
- net A4: now also D17.1 (K), D18.1 (K), D19.1 (K), D20.1 (K); no longer D16.1 (K)
- net A5: now also D21.1 (K), D22.1 (K), D23.1 (K), D24.1 (K); no longer D20.1 (K)
- net A6: now also D25.1 (K), D26.1 (K), D27.1 (K), D28.1 (K); no longer D24.1 (K)
- net A7: now also D29.1 (K), D30.1 (K), D31.1 (K), D32.1 (K); no longer D28.1 (K)
- net A8: now also D33.1 (K), D34.1 (K), D35.1 (K), D36.1 (K); no longer D32.1 (K)
- net A9: now also D37.1 (K), D38.1 (K), D39.1 (K), D40.1 (K); no longer D36.1 (K)
- net B6: no longer SW10.2, SW14.2, SW18.2, SW2.2, SW22.2, SW26.2, SW30.2, SW34.2, SW38.2, SW42.2, SW46.2, SW6.2
- net B7: now also SW10.2, SW14.2, SW18.2, SW2.2, SW22.2, SW26.2, SW30.2, SW34.2, SW38.2, SW42.2, SW46.2, SW6.2; no longer SW11.2, SW15.2, SW19.2, SW23.2, SW27.2, SW3.2, SW31.2, SW35.2, SW39.2, SW43.2, SW47.2, SW7.2
- net B8: now also SW11.2, SW15.2, SW19.2, SW23.2, SW27.2, SW3.2, SW31.2, SW35.2, SW39.2, SW43.2, SW47.2, SW7.2; no longer SW12.2, SW16.2, SW20.2, SW24.2, SW28.2, SW32.2, SW36.2, SW4.2, SW40.2, SW44.2, SW48.2, SW8.2
- net A0: now reaches D1.1 (K)
- net A0: now also D2.1 (K), D3.1 (K), D4.1 (K)
- new net 5V: J1.1 (VBUS)
- new net B9: SW12.2, SW16.2, SW20.2, SW24.2, SW28.2, SW32.2, SW36.2, SW4.2, SW40.2, SW44.2, SW48.2, SW8.2
- new net G: J1.5 (GND)
Other:
- moved on the sheet: D1, D10, D11, D12, D13, D14, D15, D16, D17, D18, D19, D2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
